File: pcb/mainboard/mainboard.kicad_pcb (KiCad board)
At the start: 2 copper layers, 139 x 190 mm, 254 parts, among them J1 PWR, J2 Conn_01x03_Male, J3 USB_B, J4 UI, J5 Conn_02x03_Odd_Even, J6 RES1, K1 EC2-12NU, K10 EC2-12NU, K11 EC2-12NU, K12 EC2-12NU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

Commit message: Update to Kicad v9, new power supply board and other modifications
Parts:
- removed LOGO1: LOGO_SH, 01_Sebastian:SebastianHarnisch
Routing:
- net unconnected-(J3-Shield-Pad5)_1: track 12.0 -> 0.00 mm
- net unconnected-(J3-Shield-Pad5): track 0.00 -> 12.0 mm
Other:
- board text added: "SEBASTIAN HARNISCH"
