File: pcb/ui_board/ui_board.kicad_pcb (KiCad board)
At the start: 2 copper layers, 212 x 67 mm, 134 parts, among them J1 PWR3.3V, J2 UI, J3 Conn_02x03_Odd_Even, Q1 BSS138, Q2 IRLML6402, Q3 IRLML6402, Q4 IRLML6402, Q5 IRLML6402, Q6 IRLML6402, Q7 IRLML6402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

Commit message: Update to Kicad v9, new power supply board and other modifications
Parts:
- removed LOGO1: LOGO_SH, 01_Sebastian:SebastianHarnisch
Other:
- board text added: "SEBASTIAN HARNISCH"
